Commit message: model_robot_ysag

File: urdf/mobile_base.xacro (robot description, xacro)
@@ -45,21 +45,6 @@
     <xacro:wheel_link prefix="right" />
     <xacro:wheel_link prefix="left" />
-    <link name="caster_wheel_link">
-        <visual>
-            <geometry>
-                <sphere radius="${wheel_radius / 2.0}" />
-            </geometry>
-            <origin xyz="0 0 0" rpy="0 0 0" />
-            <material name="grey" />
-        </visual>
-        <collision>
-            <geometry>
-                <sphere radius="${wheel_radius / 2.0}" />
-            </geometry>
-            <origin xyz="0 0 0" rpy="0 0 0" />
-        </collision>
-        <xacro:sphere_inertia m="0.5" r="${wheel_radius / 2.0}"
-                              o_xyz="0 0 0" o_rpy="0 0 0" />
-    </link>
+    <xacro:wheel_link prefix="right_front" />
+    <xacro:wheel_link prefix="left_front" />
     <joint name="base_joint" type="fixed">
         <parent link="base_footprint" />
@@ -79,8 +64,15 @@
         <axis xyz="0 1 0" />
     </joint>
-    <joint name="base_caster_wheel_joint" type="fixed">
+    <joint name="base_right_front_wheel_joint" type="continuous">
         <parent link="base_link" />
-        <child link="caster_wheel_link" />
-        <origin xyz="${base_length / 3.0} 0 ${-wheel_radius / 2.0}" rpy="0 0 0" />
+        <child link="right_front_wheel_link" />
+        <origin xyz="${base_length / 4.0} ${-(base_width + wheel_length) / 2.0} 0" rpy="0 0 0" />
+        <axis xyz="0 1 0" />
+    </joint>
+    <joint name="base_left_front_wheel_joint" type="continuous">
+        <parent link="base_link" />
+        <child link="left_front_wheel_link" />
+        <origin xyz="${base_length / 4.0} ${(base_width + wheel_length) / 2.0} 0" rpy="0 0 0" />
+        <axis xyz="0 1 0" />
     </joint>
 </robot>

File: urdf/mobile_base_gazebo.xacro (robot description, xacro)
@@ -19,8 +19,22 @@
     <gazebo>
         <plugin
+            filename="gz-sim-diff-drive-system"
+            name="gz::sim::systems::DiffDrive">
+            <left_joint>base_left_front_wheel_joint</left_joint>
+            <right_joint>base_right_front_wheel_joint</right_joint>
+            <wheel_separation>0.45</wheel_separation>
+            <wheel_radius>0.1</wheel_radius>
+            <frame_id>odom</frame_id>
+            <child_frame_id>base_footprint</child_frame_id>
+        </plugin>
+    </gazebo>
+    <gazebo>
+        <plugin
             filename="gz-sim-joint-state-publisher-system"
             name="gz::sim::systems::JointStatePublisher">
             <joint_name>base_left_wheel_joint</joint_name>
+            <joint_name>base_left_front_wheel_joint</joint_name>
             <joint_name>base_right_wheel_joint</joint_name>
+            <joint_name>base_right_front_wheel_joint</joint_name>
         </plugin>
     </gazebo>

Commit message: backversion2roda

File: urdf/mobile_base.xacro (robot description, xacro)
@@ -45,6 +45,21 @@
     <xacro:wheel_link prefix="right" />
     <xacro:wheel_link prefix="left" />
-    <xacro:wheel_link prefix="right_front" />
-    <xacro:wheel_link prefix="left_front" />
+    <link name="caster_wheel_link">
+        <visual>
+            <geometry>
+                <sphere radius="${wheel_radius / 2.0}" />
+            </geometry>
+            <origin xyz="0 0 0" rpy="0 0 0" />
+            <material name="grey" />
+        </visual>
+        <collision>
+            <geometry>
+                <sphere radius="${wheel_radius / 2.0}" />
+            </geometry>
+            <origin xyz="0 0 0" rpy="0 0 0" />
+        </collision>
+        <xacro:sphere_inertia m="0.5" r="${wheel_radius / 2.0}"
+                              o_xyz="0 0 0" o_rpy="0 0 0" />
+    </link>
     <joint name="base_joint" type="fixed">
         <parent link="base_footprint" />
@@ -64,15 +79,8 @@
         <axis xyz="0 1 0" />
     </joint>
-    <joint name="base_right_front_wheel_joint" type="continuous">
+    <joint name="base_caster_wheel_joint" type="fixed">
         <parent link="base_link" />
-        <child link="right_front_wheel_link" />
-        <origin xyz="${base_length / 4.0} ${-(base_width + wheel_length) / 2.0} 0" rpy="0 0 0" />
-        <axis xyz="0 1 0" />
-    </joint>
-    <joint name="base_left_front_wheel_joint" type="continuous">
-        <parent link="base_link" />
-        <child link="left_front_wheel_link" />
-        <origin xyz="${base_length / 4.0} ${(base_width + wheel_length) / 2.0} 0" rpy="0 0 0" />
-        <axis xyz="0 1 0" />
+        <child link="caster_wheel_link" />
+        <origin xyz="${base_length / 3.0} 0 ${-wheel_radius / 2.0}" rpy="0 0 0" />
     </joint>
 </robot>

File: urdf/mobile_base_gazebo.xacro (robot description, xacro)
@@ -19,22 +19,8 @@
     <gazebo>
         <plugin
-            filename="gz-sim-diff-drive-system"
-            name="gz::sim::systems::DiffDrive">
-            <left_joint>base_left_front_wheel_joint</left_joint>
-            <right_joint>base_right_front_wheel_joint</right_joint>
-            <wheel_separation>0.45</wheel_separation>
-            <wheel_radius>0.1</wheel_radius>
-            <frame_id>odom</frame_id>
-            <child_frame_id>base_footprint</child_frame_id>
-        </plugin>
-    </gazebo>
-    <gazebo>
-        <plugin
             filename="gz-sim-joint-state-publisher-system"
             name="gz::sim::systems::JointStatePublisher">
             <joint_name>base_left_wheel_joint</joint_name>
-            <joint_name>base_left_front_wheel_joint</joint_name>
             <joint_name>base_right_wheel_joint</joint_name>
-            <joint_name>base_right_front_wheel_joint</joint_name>
         </plugin>
     </gazebo>

Commit message: penyesuaian model robot

File: urdf/mobile_base.xacro (robot description, xacro)
@@ -1,9 +1,9 @@
 <?xml version="1.0"?>
 <robot xmlns:xacro="http://www.ros.org/wiki/xacro">
-    <xacro:property name="base_length" value="0.6" />
-    <xacro:property name="base_width" value="0.4" />
-    <xacro:property name="base_height" value="0.2" />
-    <xacro:property name="wheel_radius" value="0.1" />
-    <xacro:property name="wheel_length" value="0.05" />
+    <xacro:property name="base_length" value="0.15" />
+    <xacro:property name="base_width" value="0.15" />
+    <xacro:property name="base_height" value="0.05" />
+    <xacro:property name="wheel_radius" value="0.03" />
+    <xacro:property name="wheel_length" value="0.02" />
     <link name="base_footprint" />
     <link name="base_link">
@@ -45,5 +45,22 @@
     <xacro:wheel_link prefix="right" />
     <xacro:wheel_link prefix="left" />
-    <link name="caster_wheel_link">
+    <link name="caster_front_wheel_link">
+        <visual>
+            <geometry>
+                <sphere radius="${wheel_radius / 2.0}" />
+            </geometry>
+            <origin xyz="0 0 0" rpy="0 0 0" />
+            <material name="grey" />
+        </visual>
+        <collision>
+            <geometry>
+                <sphere radius="${wheel_radius / 2.0}" />
+            </geometry>
+            <origin xyz="0 0 0" rpy="0 0 0" />
+        </collision>
+        <xacro:sphere_inertia m="0.5" r="${wheel_radius / 2.0}"
+                              o_xyz="0 0 0" o_rpy="0 0 0" />
+    </link>
+    <link name="caster_rear_wheel_link">
         <visual>
             <geometry>
@@ -70,5 +87,5 @@
         <parent link="base_link" />
         <child link="right_wheel_link" />
-        <origin xyz="${-base_length / 4.0} ${-(base_width + wheel_length) / 2.0} 0" rpy="0 0 0" />
+        <origin xyz="${-base_length*0.0 / 4.0} ${-(base_width + wheel_length) / 2.0} 0" rpy="0 0 0" />
         <axis xyz="0 1 0" />
     </joint>
@@ -76,11 +93,16 @@
         <parent link="base_link" />
         <child link="left_wheel_link" />
-        <origin xyz="${-base_length / 4.0} ${(base_width + wheel_length) / 2.0} 0" rpy="0 0 0" />
+        <origin xyz="${-base_length*0.0 / 4.0} ${(base_width + wheel_length) / 2.0} 0" rpy="0 0 0" />
         <axis xyz="0 1 0" />
     </joint>
-    <joint name="base_caster_wheel_joint" type="fixed">
+    <joint name="base_caster_front_wheel_joint" type="fixed">
         <parent link="base_link" />
-        <child link="caster_wheel_link" />
+        <child link="caster_front_wheel_link" />
         <origin xyz="${base_length / 3.0} 0 ${-wheel_radius / 2.0}" rpy="0 0 0" />
     </joint>
+    <joint name="base_caster_rear_wheel_joint" type="fixed">
+        <parent link="base_link" />
+        <child link="caster_rear_wheel_link" />
+        <origin xyz="${-base_length / 3.0} 0 ${-wheel_radius / 2.0}" rpy="0 0 0" />
+    </joint>
 </robot>
